File: hardware/keyboard-cherry-mx-pcb-mounted/GestureSensor.sch (KiCad schematic (older format))
At the start: 0 parts

Commit message: Adds STM32F413 to cherry mx pcb mounted board.
Parts:
- added U? (x2): APDS-9960, QFN_DS-9930, symbol Sij_Sensors:APDS-9930
Changed lines of the file:
@@
 $Descr A4 11693 8268
 encoding utf-8
-Sheet 9 9
+Sheet 9 10
 Title ""
 Date ""
@@
 Comment4 ""
 $EndDescr
+$Comp
+L Sij_Sensors:APDS-9930 U?
+U 1 1 5E817D7C
+P 4500 3300
+F 0 "U?" H 4650 2850 60  0000 C CNN
+F 1 "APDS-9960" H 4650 2750 60  0000 C CNN
+F 2 "QFN_DS-9930" H 5300 3540 60  0001 C CNN
+F 3 "" H 4500 3300 60  0000 C CNN
+	1    4500 3300
+	1    0    0    -1
+$EndComp
+$Comp
+L Sij_Sensors:APDS-9930 U?
+U 1 1 5E81B7BE
+P 4500 4500
+F 0 "U?" H 4650 4050 60  0000 C CNN
+F 1 "APDS-9960" H 4650 3950 60  0000 C CNN
+F 2 "QFN_DS-9930" H 5300 4740 60  0001 C CNN
+F 3 "" H 4500 4500 60  0000 C CNN
+	1    4500 4500
+	1    0    0    -1
+$EndComp
 $EndSCHEMATC
