File: hardware/keyboard-cherry-mx-pcb-mounted/keyboard-cherry-mx-pcb-mounted.kicad_pcb (KiCad board)
At the start: 2 copper layers, 159 parts, among them SW1 ESC, SW10 F12, SW11 F5, SW12 Delete, SW13 F6, SW14 F7, SW15 `, SW16 8, SW17 1, SW18 9, SW19 2, SW2 F8, SW20 0, SW21 3, SW22 -, SW23 4, SW24 =, SW25 5, SW26 Backspace, SW27 6, SW28 Home, SW29 7, SW3 F1, SW30 Ctrl, SW32 Workspace, SW34 Alt, SW36 Space, SW38 Left Arrow, SW4 F9, SW40 Down Arrow, SW42 Right Arrow, SW46 LShift, SW47 ,, SW48 z, SW49 ., SW5 F2, SW50 x, SW51 /, SW52 c, SW53 RShift, SW54 v, SW55 Up Arrow, SW56 b, SW57 End, SW58 n, SW59 m, SW6 F10, SW60 Caps lock, SW61 k, SW62 a, SW63 l, SW64 s, SW65 ;, SW66 d, SW67 ', SW68 f, SW69 Enter, SW7 F3, SW70 g, SW71 PgDn, SW72 h, SW73 j, SW74 Tab, SW75 i, SW76 q, SW77 o, SW78 w, SW79 p, SW8 F11, SW80 e, SW81 [, SW82 r, SW83 ], SW84 t, SW85 \, SW86 y, SW87 PgUp, SW88 u, SW9 F4, U1 BGM13S

Commit message: Adds completed sensor and power connections. Still need to add USB footprint then sch are done for version 1.0
Parts:
- removed the SW38 at (317.5, 492.9)
- added C1: 4.7u, Capacitor_SMD:C_0805_2012Metric, F.Cu at (278.0, 616.0)
- added C10: 1u, Capacitor_SMD:C_0805_2012Metric, F.Cu at (273.6, 616.0)
- added C2: 0.1u, Capacitor_SMD:C_0805_2012Metric, F.Cu at (289.3, 601.5)
- added C3: 0.1u, Capacitor_SMD:C_0805_2012Metric, F.Cu at (293.8, 601.5)
- added C4: 15pF, Capacitor_SMD:C_0805_2012Metric, F.Cu at (286.8, 610.6)
- added C5: 0.1u, Capacitor_SMD:C_0805_2012Metric, F.Cu at (292.6, 604.5)
- added C6: 15pF, Capacitor_SMD:C_0805_2012Metric, F.Cu at (282.4, 613.6)
- added C7: 4.7u, Capacitor_SMD:C_0805_2012Metric, F.Cu at (288.2, 606.3)
- added C8: 0.1u, Capacitor_SMD:C_0805_2012Metric, F.Cu at (282.4, 616.5)
- added C9: 0.1u, Capacitor_SMD:C_0805_2012Metric, F.Cu at (282.4, 610.6)
- added D34: 1N4148W, Diode_SMD:D_SOD-123, F.Cu at (274.4, 594.8)
- added D35: 1N4148W, Diode_SMD:D_SOD-123, F.Cu at (268.6, 594.8)
- added JP1: BootJumper, Jumper:SolderJumper-3_P1.3mm_Bridged12_Pad1.0x1.5mm, F.Cu at (268.6, 616.3)
- added R1: 10k, Resistor_SMD:R_0805_2012Metric, F.Cu at (322.3, 574.4)
- added R2: 4.7k, Resistor_SMD:R_0805_2012Metric, F.Cu at (322.3, 577.4)
- added R3: 4.7k, Resistor_SMD:R_0805_2012Metric, F.Cu at (326.7, 574.4)
- added R4: 4.7k, Resistor_SMD:R_0805_2012Metric, F.Cu at (322.3, 580.3)
- added R5: 4.7k, Resistor_SMD:R_0805_2012Metric, F.Cu at (326.7, 577.4)
- added R6: 4.7k, Resistor_SMD:R_0805_2012Metric, F.Cu at (322.3, 583.3)
- added R7: 4.7k, Resistor_SMD:R_0805_2012Metric, F.Cu at (326.7, 580.3)
- added R8: 5.1k, Resistor_SMD:R_0805_2012Metric, F.Cu at (304.0, 601.5)
- added R9: 5.1k, Resistor_SMD:R_0805_2012Metric, F.Cu at (308.4, 601.5)
- added SW1: RST, Button_Switch_SMD:SW_SPST_B3U-1000P, F.Cu at (283.1, 607.0)
- added SW35: Alt, Button_Switch_Keyboard:SW_Cherry_MX_1.50u_PCB, F.Cu at (278.4, 578.0)
- added SW36: Ctrl, Button_Switch_Keyboard:SW_Cherry_MX_1.50u_PCB, F.Cu at (298.6, 578.0)
- added SW37: Left Arrow, Button_Switch_Keyboard:SW_Cherry_MX_1.00u_PCB, F.Cu at (317.5, 492.9)
- added U2: TCA9543, Package_SO:SOIC-14_3.9x8.7mm_P1.27mm, F.Cu at (315.8, 578.1)
- added Y1: 8MHz, Crystal:Crystal_SMD_TXC_7A-2Pin_5x3.2mm, F.Cu at (283.7, 602.5)
- U1: value BGM13S -> STM32F413RHTx; footprint Sij_MCU:BGM13S -> Package_QFP:LQFP-64_10x10mm_P0.5mm
- moved U1 431.9 mm to (273.0, 607.3)
- renumbered D32 to D31, D34 to D32, D36 to D33, D38 to D36, D40 to D37, D42 to D38, D46 to D39, D47 to D40, D48 to D41, D49 to D42, D50 to D43, D51 to D44, D52 to D45, D53 to D46, D54 to D47, D55 to D48, D56 to D49, D57 to D50, D58 to D51, D59 to D52, D60 to D53, D61 to D54, D62 to D55, D63 to D56, D64 to D57, D65 to D58, D66 to D59, D67 to D60, D68 to D61, D69 to D62, D70 to D63, D71 to D64, D72 to D65, D73 to D66, D74 to D67, D75 to D68, D76 to D69, D77 to D70, D78 to D71, D79 to D72, D80 to D73, D81 to D74, D82 to D75, D83 to D76, D84 to D77, D85 to D78, D86 to D79, D87 to D80, D88 to D81, SW9 to SW10, SW10 to SW11, SW11 to SW12, SW12 to SW13, SW13 to SW14, SW14 to SW15, SW15 to SW16, SW16 to SW17, SW17 to SW18, SW18 to SW19, SW1 to SW2, SW19 to SW20, SW20 to SW21, SW21 to SW22, SW22 to SW23, SW23 to SW24, SW24 to SW25, SW25 to SW26, SW26 to SW27, SW27 to SW28, SW28 to SW29, SW2 to SW3, SW29 to SW30, SW30 to SW31, SW34 to SW33, SW36 to SW34, SW40 to SW38, SW42 to SW39, SW3 to SW4, SW46 to SW40, SW47 to SW41, SW48 to SW42, SW49 to SW43, SW50 to SW44, SW51 to SW45, SW52 to SW46, SW53 to SW47, SW54 to SW48, SW55 to SW49, SW4 to SW5, SW56 to SW50, SW57 to SW51, SW58 to SW52, SW59 to SW53, SW60 to SW54, SW61 to SW55, SW62 to SW56, SW63 to SW57, SW64 to SW58, SW65 to SW59, SW5 to SW6, SW66 to SW60, SW67 to SW61, SW68 to SW62, SW69 to SW63, SW70 to SW64, SW71 to SW65, SW72 to SW66, SW73 to SW67, SW74 to SW68, SW75 to SW69, SW6 to SW7, SW76 to SW70, SW77 to SW71, SW78 to SW72, SW79 to SW73, SW80 to SW74, SW81 to SW75, SW82 to SW76, SW83 to SW77, SW84 to SW78, SW85 to SW79, SW7 to SW8, SW86 to SW80, SW87 to SW81, SW88 to SW82, SW8 to SW9
Connections:
- net /SWO renamed Net-(U1-Pad29)
- D1 pad 1: /KeySwitches/Row0/C0 -> /C0
- D10 pad 1: /KeySwitches/Row0/C12 -> /C12
- D11 pad 1: /KeySwitches/Row0/C5 -> /C5
- D12 pad 1: /KeySwitches/Row0/C13 -> /C13
- D13 pad 1: /KeySwitches/Row0/C6 -> /C6
- D14 pad 1: /KeySwitches/Row0/C7 -> /C7
- D15 pad 1: /KeySwitches/Row0/C0 -> /C0
- D16 pad 1: /KeySwitches/Row0/C8 -> /C8
- D17 pad 1: /KeySwitches/Row0/C1 -> /C1
- D18 pad 1: /KeySwitches/Row0/C9 -> /C9
- D19 pad 1: /KeySwitches/Row0/C2 -> /C2
- D2 pad 1: /KeySwitches/Row0/C8 -> /C8
- D20 pad 1: /KeySwitches/Row0/C10 -> /C10
- D21 pad 1: /KeySwitches/Row0/C3 -> /C3
- D22 pad 1: /KeySwitches/Row0/C11 -> /C11
- D23 pad 1: /KeySwitches/Row0/C4 -> /C4
- D24 pad 1: /KeySwitches/Row0/C12 -> /C12
- D25 pad 1: /KeySwitches/Row0/C5 -> /C5
- D26 pad 1: /KeySwitches/Row0/C13 -> /C13
- D27 pad 1: /KeySwitches/Row0/C6 -> /C6
- D28 pad 1: /KeySwitches/Row1/C14 -> /C14
- D29 pad 1: /KeySwitches/Row0/C7 -> /C7
- D3 pad 1: /KeySwitches/Row0/C1 -> /C1
- D30 pad 1: /KeySwitches/Row0/C0 -> /C0
- D31 pad 1: /KeySwitches/Row0/C1 -> /C1
- D32 pad 1: /KeySwitches/Row0/C2 -> /C2
- D33 pad 1: /KeySwitches/Row0/C3 -> /C3
- D36 pad 1: /KeySwitches/Row0/C4 -> /C6
- D37 pad 1: /KeySwitches/Row0/C5 -> /C7
- D38 pad 1: /KeySwitches/Row0/C6 -> /C8
- D39 pad 1: /KeySwitches/Row0/C0 -> /C0
- D4 pad 1: /KeySwitches/Row0/C9 -> /C9
- D40 pad 1: /KeySwitches/Row0/C8 -> /C8
- D41 pad 1: /KeySwitches/Row0/C1 -> /C1
- D42 pad 1: /KeySwitches/Row0/C9 -> /C9
- D43 pad 1: /KeySwitches/Row0/C2 -> /C2
- D44 pad 1: /KeySwitches/Row0/C10 -> /C10
- D45 pad 1: /KeySwitches/Row0/C3 -> /C3
- D46 pad 1: /KeySwitches/Row0/C11 -> /C11
- D47 pad 1: /KeySwitches/Row0/C4 -> /C4
- D48 pad 1: /KeySwitches/Row0/C12 -> /C12
- D49 pad 1: /KeySwitches/Row0/C5 -> /C5
- D5 pad 1: /KeySwitches/Row0/C2 -> /C2
- D50 pad 1: /KeySwitches/Row0/C13 -> /C13
- D51 pad 1: /KeySwitches/Row0/C6 -> /C6
- D52 pad 1: /KeySwitches/Row0/C7 -> /C7
- D53 pad 1: /KeySwitches/Row0/C0 -> /C0
- D54 pad 1: /KeySwitches/Row0/C8 -> /C8
- D55 pad 1: /KeySwitches/Row0/C1 -> /C1
- D56 pad 1: /KeySwitches/Row0/C9 -> /C9
- D57 pad 1: /KeySwitches/Row0/C2 -> /C2
- D58 pad 1: /KeySwitches/Row0/C10 -> /C10
- D59 pad 1: /KeySwitches/Row0/C3 -> /C3
- D6 pad 1: /KeySwitches/Row0/C10 -> /C10
- D60 pad 1: /KeySwitches/Row0/C11 -> /C11
- D61 pad 1: /KeySwitches/Row0/C4 -> /C4
- D62 pad 1: /KeySwitches/Row0/C12 -> /C12
- D63 pad 1: /KeySwitches/Row0/C5 -> /C5
- D64 pad 1: /KeySwitches/Row0/C13 -> /C13
- D65 pad 1: /KeySwitches/Row0/C6 -> /C6
- D66 pad 1: /KeySwitches/Row0/C7 -> /C7
- D67 pad 1: /KeySwitches/Row0/C0 -> /C0
- D68 pad 1: /KeySwitches/Row0/C8 -> /C8
- D69 pad 1: /KeySwitches/Row0/C1 -> /C1
- D7 pad 1: /KeySwitches/Row0/C3 -> /C3
- D70 pad 1: /KeySwitches/Row0/C9 -> /C9
- D71 pad 1: /KeySwitches/Row0/C2 -> /C2
- D72 pad 1: /KeySwitches/Row0/C10 -> /C10
- D73 pad 1: /KeySwitches/Row0/C3 -> /C3
- D74 pad 1: /KeySwitches/Row0/C11 -> /C11
- D75 pad 1: /KeySwitches/Row0/C4 -> /C4
- D76 pad 1: /KeySwitches/Row0/C12 -> /C12
- D77 pad 1: /KeySwitches/Row0/C5 -> /C5
- D78 pad 1: /KeySwitches/Row0/C13 -> /C13
- D79 pad 1: /KeySwitches/Row0/C6 -> /C6
- D8 pad 1: /KeySwitches/Row0/C11 -> /C11
- D80 pad 1: /KeySwitches/Row1/C14 -> /C14
- D81 pad 1: /KeySwitches/Row0/C7 -> /C7
- D9 pad 1: /KeySwitches/Row0/C4 -> /C4
- SW10 pad 1: /KeySwitches/R0 -> /R0
- SW11 pad 1: /KeySwitches/R0 -> /R0
- SW12 pad 1: /KeySwitches/R0 -> /R0
- SW13 pad 1: /KeySwitches/R0 -> /R0
- SW14 pad 1: /KeySwitches/R0 -> /R0
- SW15 pad 1: /KeySwitches/R0 -> /R0
- SW16 pad 1: /KeySwitches/R1 -> /R1
- SW17 pad 1: /KeySwitches/R1 -> /R1
- SW18 pad 1: /KeySwitches/R1 -> /R1
- SW19 pad 1: /KeySwitches/R1 -> /R1
- SW2 pad 1: /KeySwitches/R0 -> /R0
- SW20 pad 1: /KeySwitches/R1 -> /R1
- SW21 pad 1: /KeySwitches/R1 -> /R1
- SW22 pad 1: /KeySwitches/R1 -> /R1
- SW23 pad 1: /KeySwitches/R1 -> /R1
- SW24 pad 1: /KeySwitches/R1 -> /R1
- SW25 pad 1: /KeySwitches/R1 -> /R1
- SW26 pad 1: /KeySwitches/R1 -> /R1
- SW27 pad 1: /KeySwitches/R1 -> /R1
- SW28 pad 1: /KeySwitches/R1 -> /R1
- SW29 pad 1: /KeySwitches/R1 -> /R1
- SW3 pad 1: /KeySwitches/R0 -> /R0
- SW30 pad 1: /KeySwitches/R1 -> /R1
- SW31 pad 1: /KeySwitches/R5 -> /R5
- SW32 pad 1: /KeySwitches/R5 -> /R5
- SW33 pad 1: /KeySwitches/R5 -> /R5
- SW34 pad 1: /KeySwitches/R5 -> /R5
- SW38 pad 1: /KeySwitches/R5 -> /R5
- SW39 pad 1: /KeySwitches/R5 -> /R5
- SW4 pad 1: /KeySwitches/R0 -> /R0
- SW40 pad 1: /KeySwitches/R4 -> /R4
- SW41 pad 1: /KeySwitches/R4 -> /R4
- SW42 pad 1: /KeySwitches/R4 -> /R4
- SW43 pad 1: /KeySwitches/R4 -> /R4
- SW44 pad 1: /KeySwitches/R4 -> /R4
- SW45 pad 1: /KeySwitches/R4 -> /R4
- SW46 pad 1: /KeySwitches/R4 -> /R4
- SW47 pad 1: /KeySwitches/R4 -> /R4
- SW48 pad 1: /KeySwitches/R4 -> /R4
- SW49 pad 1: /KeySwitches/R4 -> /R4
- SW5 pad 1: /KeySwitches/R0 -> /R0
- SW50 pad 1: /KeySwitches/R4 -> /R4
- SW51 pad 1: /KeySwitches/R4 -> /R4
- SW52 pad 1: /KeySwitches/R4 -> /R4
- SW53 pad 1: /KeySwitches/R4 -> /R4
- SW54 pad 1: /KeySwitches/R3 -> /R3
- SW55 pad 1: /KeySwitches/R3 -> /R3
- SW56 pad 1: /KeySwitches/R3 -> /R3
- SW57 pad 1: /KeySwitches/R3 -> /R3
- SW58 pad 1: /KeySwitches/R3 -> /R3
- SW59 pad 1: /KeySwitches/R3 -> /R3
- SW6 pad 1: /KeySwitches/R0 -> /R0
- SW60 pad 1: /KeySwitches/R3 -> /R3
- SW61 pad 1: /KeySwitches/R3 -> /R3
- SW62 pad 1: /KeySwitches/R3 -> /R3
- SW63 pad 1: /KeySwitches/R3 -> /R3
- SW64 pad 1: /KeySwitches/R3 -> /R3
- SW65 pad 1: /KeySwitches/R3 -> /R3
- SW66 pad 1: /KeySwitches/R3 -> /R3
- SW67 pad 1: /KeySwitches/R3 -> /R3
- SW68 pad 1: /KeySwitches/R2 -> /R2
- SW69 pad 1: /KeySwitches/R2 -> /R2
- SW7 pad 1: /KeySwitches/R0 -> /R0
- SW70 pad 1: /KeySwitches/R2 -> /R2
- SW71 pad 1: /KeySwitches/R2 -> /R2
- SW72 pad 1: /KeySwitches/R2 -> /R2
- SW73 pad 1: /KeySwitches/R2 -> /R2
- SW74 pad 1: /KeySwitches/R2 -> /R2
- SW75 pad 1: /KeySwitches/R2 -> /R2
- SW76 pad 1: /KeySwitches/R2 -> /R2
- SW77 pad 1: /KeySwitches/R2 -> /R2
- SW78 pad 1: /KeySwitches/R2 -> /R2
- SW79 pad 1: /KeySwitches/R2 -> /R2
- SW8 pad 1: /KeySwitches/R0 -> /R0
- SW80 pad 1: /KeySwitches/R2 -> /R2
- SW81 pad 1: /KeySwitches/R2 -> /R2
- SW82 pad 1: /KeySwitches/R2 -> /R2
- SW9 pad 1: /KeySwitches/R0 -> /R0
- U1 pad 1: GND -> +3V3
- U1 pad 10: Net-(U1-Pad10) -> /C2
- U1 pad 11: Net-(U1-Pad11) -> /C3
- U1 pad 12: Net-(U1-Pad12) -> GND
- U1 pad 13: /R0 -> +3V3
- U1 pad 14: /R1 -> /R0
- U1 pad 15: /R2 -> /R1
- U1 pad 16: /R3 -> /R2
- U1 pad 17: /R4 -> /R3
- U1 pad 18: /R5 -> GND
- U1 pad 19: /C4 -> +3V3
- U1 pad 2: Net-(U1-Pad2) -> /C13
- U1 pad 20: GND -> /R4
- U1 pad 21: /C3 -> /R5
- U1 pad 22: +3V3 -> Net-(U1-Pad22)
- U1 pad 24: +3V3 -> /C4
- U1 pad 25: Net-(U1-Pad25) -> /C5
- U1 pad 26: /C10 -> Net-(U1-Pad26)
- U1 pad 27: /C11 -> Net-(U1-Pad27)
- U1 pad 28: /C12 -> Net-(U1-Pad28)
- U1 pad 3: Net-(U1-Pad2) -> /C14
- U1 pad 30: /C13 -> Net-(C1-Pad2)
- U1 pad 32: /C14 -> +3V3
- U1 pad 33: /C15 -> Net-(U1-Pad33)
- U1 pad 34: /SWCLK -> Net-(U1-Pad34)
- U1 pad 35: /SWDIO -> Net-(U1-Pad35)
- U1 pad 36: /C2 -> Net-(U1-Pad36)
- U1 pad 37: /C1 -> /C6
- U1 pad 38: /C0 -> /C7
- U1 pad 39: /C5 -> /C8
- U1 pad 4: GND -> /C15
- U1 pad 40: /C6 -> /C9
- U1 pad 41: /C7 -> Net-(U1-Pad41)
- U1 pad 42: /C8 -> +5V
- U1 pad 43: /C9 -> Net-(U1-Pad43)
- U1 pad 44: /~nRST -> /D-
- U1 pad 45: GND -> /D+
- U1 pad 46: GND -> /SWDIO
- U1 pad 48: GND -> +3V3
- U1 pad 49: GND -> /SWCLK
- U1 pad 5: GND -> /OSC_IN
- U1 pad 50: GND -> Net-(U1-Pad50)
- U1 pad 51: GND -> /C10
- U1 pad 6: Net-(U1-Pad6) -> /OSC_OUT
- U1 pad 7: Net-(U1-Pad7) -> /~nRST
- U1 pad 8: Net-(U1-Pad8) -> /C0
- U1 pad 9: Net-(U1-Pad9) -> /C1

Commit message: All keys except for function key row are laid out to their exact locations.
Parts:
- added C11: 0.1u, Capacitor_SMD:C_0805_2012Metric, F.Cu at (190.6, 306.0)
- added C12: 0.1u, Capacitor_SMD:C_0805_2012Metric, F.Cu at (199.0, 300.2)
- added C13: 0.1u, Capacitor_SMD:C_0805_2012Metric, F.Cu at (195.0, 306.0)
- added C14: 10u, Capacitor_SMD:C_0805_2012Metric, F.Cu at (174.3, 308.5)
- added C15: 10u, Capacitor_SMD:C_0805_2012Metric, F.Cu at (178.7, 308.5)
- added D82: Blue, LED_SMD:LED_0805_2012Metric, F.Cu at (307.0, 315.0)
- added J1: USB_C_Receptacle_USB2.0, Sij_Connectors:USB_C_Receptacle_Wurth_632723100021, F.Cu at (166.8, 304.8)
- added J2: SWDConn, Connector:Tag-Connect_TC2050-IDC-NL_2x05_P1.27mm_Vertical, F.Cu at (166.8, 317.7)
- added R10: 325, Resistor_SMD:R_0805_2012Metric, F.Cu at (183.1, 308.5)
- added U3: APDS-9960, Sij_Sensors:APDS-9930, F.Cu at (190.5, 301.7)
- added U4: APDS-9960, Sij_Sensors:APDS-9930, F.Cu at (194.7, 301.7)
- added U5: NCP1117-3.3_SOT223, Package_TO_SOT_SMD:SOT-223-3_TabPin2, F.Cu at (177.0, 302.9)
- added U6: TPD2EUSB30, Package_TO_SOT_SMD:Texas_DRT-3, F.Cu at (183.3, 300.0)
- moved SW35 114.5 mm to (204.8, 490.2)
- moved SW36 109.3 mm to (233.4, 490.2)
- moved SW29 69.4 mm to (295.3, 414.0)
- moved SW81 69.3 mm to (295.3, 433.1)
- moved SW65 69.3 mm to (295.3, 452.1)
- moved SW51 69.3 mm to (295.3, 471.2)
- moved SW13 69.3 mm to (295.3, 384.8)
- moved SW11 64.6 mm to (268.0, 384.8)
- moved SW9 63.6 mm to (248.9, 384.8)
- moved SW7 62.7 mm to (229.9, 384.8)
- moved SW39 62.3 mm to (295.3, 490.2)
- moved SW5 61.7 mm to (210.8, 384.8)
- moved SW38 61.4 mm to (276.2, 490.2)
- moved SW49 61.3 mm to (276.2, 471.2)
- moved SW37 60.4 mm to (257.2, 490.2)
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Connections:
- net /C15 renamed Net-(U1-Pad4)
- net Net-(C1-Pad2) renamed /VCAP1
- C9 pad 2: /~NRST -> /~nRST
- R1 pad 2: /PB3 -> /PB8
- SW1 pad 1: /~NRST -> /~nRST
- SW35 pad 1: Net-(SW35-Pad1) -> /R5
- SW36 pad 1: Net-(SW36-Pad1) -> /R5
- U1 pad 55: /PB3 -> /SWO
- U1 pad 61: Net-(U1-Pad61) -> /PB8
- U2 pad 3: /PB3 -> /PB8
