File: hardware/keyboard-cherry-mx-pcb-mounted/keyboard-cherry-mx-pcb-mounted.kicad_pcb (KiCad board)
At the start: 2 copper layers, 199 parts, among them J1 USB_C_Receptacle_USB2.0, J2 SWDConn, SW1 RST, SW10 F4, SW11 F12, SW12 F5, SW13 Delete, SW14 F6, SW15 F7, SW16 `, SW17 8, SW18 1, SW19 9, SW2 ESC, SW20 2, SW21 0, SW22 3, SW23 -, SW24 4, SW25 =, SW26 5, SW27 Backspace, SW28 6, SW29 Home, SW3 F8, SW30 7, SW31 Ctrl, SW32 Workspace, SW33 Alt, SW34 Space, SW35 Alt, SW36 Ctrl, SW37 Left Arrow, SW38 Down Arrow, SW39 Right Arrow, SW4 F1, SW40 LShift, SW41 ,, SW42 z, SW43 ., SW44 x, SW45 /, SW46 c, SW47 RShift, SW48 v, SW49 Up Arrow, SW5 F9, SW50 b, SW51 End, SW52 n, SW53 m, SW54 Caps lock, SW55 k, SW56 a, SW57 l, SW58 s, SW59 ;, SW6 F2, SW60 d, SW61 ', SW62 f, SW63 Enter, SW64 g, SW65 PgDn, SW66 h, SW67 j, SW68 Tab, SW69 i, SW7 F10, SW70 q, SW71 o, SW72 w, SW73 p, SW74 e, SW75 [, SW76 r, SW77 ], SW78 t, SW79 \, SW8 F3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

Commit message: Adds final key caps layout of a 75 keyboard.
Parts:
- moved SW31 338.2 mm to (27.8, 152.4)
- moved SW32 338.2 mm to (51.6, 152.4)
- moved SW33 338.2 mm to (75.4, 152.4)
- moved SW34 338.2 mm to (146.8, 152.4)
- moved SW35 338.2 mm to (220.7, 152.4)
- moved SW36 338.2 mm to (249.2, 152.4)
- moved SW37 338.2 mm to (273.1, 152.4)
- moved SW38 338.2 mm to (292.1, 152.4)
- moved SW39 338.2 mm to (311.1, 152.4)
- moved SW40 338.2 mm to (37.3, 133.3)
- moved SW41 338.2 mm to (201.6, 133.3)
- moved SW42 338.2 mm to (68.3, 133.3)
- moved SW43 338.2 mm to (220.7, 133.3)
- moved SW44 338.2 mm to (87.3, 133.3)
- moved SW45 338.2 mm to (239.7, 133.3)
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
Commit message: Adds board outline for the cherry mx pcb mounted keyboard.
Parts:
- moved C6 610.7 mm to (-178.0, 212.3)
- moved D34 610.7 mm to (-186.0, 193.5)
- moved D35 610.7 mm to (-191.8, 193.5)
- moved D39 610.7 mm to (-42.3, 128.9)
- moved D41 610.7 mm to (-48.0, 128.9)
- moved D52 610.7 mm to (-48.0, 138.9)
- moved R4 610.7 mm to (-138.1, 179.0)
- moved R7 610.7 mm to (-133.7, 179.0)
- moved Y1 610.7 mm to (-176.7, 201.1)
- moved C1 610.7 mm to (-182.4, 214.7)
- moved C10 610.7 mm to (-186.8, 214.7)
- moved C2 610.7 mm to (-171.0, 200.2)
- moved C3 610.7 mm to (-166.6, 200.2)
- moved C4 610.7 mm to (-173.6, 209.3)
- moved C5 610.7 mm to (-167.7, 203.2)
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Other:
- board outline added: 304.8 x 123.8 mm

Commit message: Adds more gesture sensors to the cherry mx pcb mounted keyboard.
Parts:
- D1, D10, D11, D12, D13, D14, D2, D3, D4, D5, D50, D6, D67, D7, D8, D9: moved to B.Cu
- moved D12 478.4 mm to (308.6, 57.1), turned to 180 degrees
- moved D10 450.2 mm to (280.0, 57.1), turned to 180 degrees
- moved D8 446.0 mm to (261.0, 57.1), turned to 180 degrees
- moved D6 406.8 mm to (241.9, 57.1), turned to 180 degrees
- moved D4 388.2 mm to (222.9, 57.1), turned to 180 degrees
- moved D2 366.4 mm to (194.3, 57.1), turned to 180 degrees
- moved D50 351.1 mm to (308.6, 142.9), turned to 180 degrees
- moved D14 345.2 mm to (175.3, 57.1), turned to 180 degrees
- moved D13 320.5 mm to (156.2, 57.1), turned to 180 degrees
- moved D11 301.9 mm to (137.2, 57.1), turned to 180 degrees
- moved D9 274.0 mm to (108.6, 57.1), turned to 180 degrees
- moved D7 261.3 mm to (89.5, 57.1), turned to 180 degrees
- moved D5 243.1 mm to (70.5, 57.1), turned to 180 degrees
- moved D3 225.1 mm to (51.4, 57.1), turned to 180 degrees
- moved D1 191.7 mm to (22.9, 57.1), turned to 180 degrees
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
Commit message: Places diodes at respective locations on cherry mx pcb mounted keyboard.
Parts:
- added C16: 0.1u, Capacitor_SMD:C_0805_2012Metric, F.Cu at (-127.2, 68.9)
- added C17: 0.1u, Capacitor_SMD:C_0805_2012Metric, F.Cu at (-122.8, 68.9)
- added R11: 1k, Resistor_SMD:R_0805_2012Metric, F.Cu at (-127.2, 71.9)
- added R12: 1k, Resistor_SMD:R_0805_2012Metric, F.Cu at (-122.8, 71.9)
- added R13: 1k, Resistor_SMD:R_0805_2012Metric, F.Cu at (-127.2, 74.8)
- added R14: 1k, Resistor_SMD:R_0805_2012Metric, F.Cu at (-122.8, 74.8)
- added U7: APDS-9960, Sij_Sensors:APDS-9930, F.Cu at (-131.5, 70.3)
- added U8: APDS-9960, Sij_Sensors:APDS-9930, F.Cu at (-131.5, 76.1)
- D15, D16, D17, D18, D19, D20, D21, D22, D23, D24, D25, D26, D27, D28, D29, D30, D31, D32, D33, D34, D35, D36, D37, D38, D39, D40, D41, D42, D43, D44, D45, D46, D47, D48, D49, D51, D52, D53, D54, D55, D56, D57, D58, D59, D60, D61, D62, D63, D64, D65, D66, D68, D69, D70, D71, D72, D73, D74, D75, D76, D77, D78, D79, D80, D81: moved to B.Cu
- R2, R3, R4, R5, R6, R7: value 4.7k -> 1k
- U2: value TCA9543 -> PCA9546AD; footprint Package_SO:SOIC-14_3.9x8.7mm_P1.27mm -> Package_SO:SOIC-16_3.9x9.9mm_P1.27mm
- moved D48 563.0 mm to (289.6, 142.9), turned to 180 degrees
- moved D46 525.4 mm to (263.4, 142.9), turned to 180 degrees
- moved D44 487.9 mm to (237.2, 142.9), turned to 180 degrees
- moved D42 457.4 mm to (218.1, 142.9), turned to 180 degrees
- moved D40 455.7 mm to (199.1, 142.9), turned to 180 degrees
- moved D35 439.6 mm to (246.7, 161.9), turned to 180 degrees
- moved D62 431.8 mm to (277.7, 123.8), turned to 180 degrees
- moved D60 418.9 mm to (246.7, 123.8), turned to 180 degrees
- moved D34 405.4 mm to (218.1, 161.9), turned to 180 degrees
- moved D80 401.0 mm to (308.6, 104.8), turned to 180 degrees
- moved D28 399.4 mm to (308.6, 85.7), turned to 180 degrees
- moved C9 394.7 mm to (189.7, 352.8)
- moved C1 394.7 mm to (185.3, 358.2)
- moved C10 394.7 mm to (180.9, 358.2)
- moved C2 394.7 mm to (196.6, 343.7)
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Connections:
- R1 pad 2: /PB8 -> /PB10
- U1 pad 29: Net-(U1-Pad29) -> /PB10
- U1 pad 33: Net-(U1-Pad33) -> /PB12
- U1 pad 34: Net-(U1-Pad34) -> /PB13
- U1 pad 35: Net-(U1-Pad35) -> /PB14
- U1 pad 36: Net-(U1-Pad36) -> /PB15
- U1 pad 56: /PB4 -> Net-(U1-Pad56)
- U1 pad 57: /PB5 -> Net-(U1-Pad57)
- U1 pad 61: /PB8 -> Net-(U1-Pad61)
- U2 pad 10: Net-(R5-Pad2) -> Net-(R11-Pad2)
- U2 pad 12: /I2C1_SCL -> Net-(R12-Pad2)
- U2 pad 13: /I2C1_SDA -> GND
- U2 pad 14: +3V3 -> /I2C1_SDA
- U2 pad 3: /PB8 -> /PB10
- U2 pad 4: Net-(U2-Pad4) -> Net-(R6-Pad2)
- U2 pad 5: Net-(R6-Pad2) -> Net-(R4-Pad2)
- U2 pad 6: Net-(R4-Pad2) -> Net-(R7-Pad2)
- U2 pad 7: GND -> Net-(R5-Pad2)
- U2 pad 8: Net-(U2-Pad8) -> GND
- U2 pad 9: Net-(R7-Pad2) -> Net-(R13-Pad2)
- U3 pad 2: /PB4 -> /PB12
- U4 pad 2: /PB5 -> /PB13

Commit message: Aligns the keys so the column connections are more consistent. e.g. right most keys will have same column connection.
Parts:
- removed the C1 at (185.3, 358.2)
- removed the C4 at (194.1, 352.8)
- added C5: 0.1u, Capacitor_SMD:C_0805_2012Metric, F.Cu at (-43.2, 213.4)
- added C7: 15pF, Capacitor_SMD:C_0805_2012Metric, F.Cu at (-51.4, 208.3)
- C10: value 1u -> 4.7u
- C6: value 15pF -> 1u
- C8: value 0.1u -> 15pF
- moved C9 290.0 mm to (-50.2, 189.9)
- moved SW1 286.8 mm to (-50.2, 193.0), turned to 180 degrees
- moved C8 282.2 mm to (-51.4, 212.1), turned to 180 degrees
- moved C2 275.9 mm to (-39.4, 208.3), turned to 90 degrees
- moved Y1 272.7 mm to (-46.4, 210.2), turned to 270 degrees
- moved C1 271.0 mm to (-34.3, 201.9), turned to 180 degrees
- moved C6 270.3 mm to (-40.0, 213.4), turned to 270 degrees
- moved C3 265.3 mm to (-33.7, 221.0)
- moved JP1 263.2 mm to (-32.4, 197.5)
- moved C4 257.9 mm to (-21.0, 208.3), turned to 90 degrees
- moved R13 253.3 mm to (4.45, 197.5)
- moved R14 251.9 mm to (4.85, 205.9)
- moved U1 251.9 mm to (-30.6, 211.7)
- moved C10 248.6 mm to (-26.4, 221.0), turned to 180 degrees
- renumbered C2 to C1, C16 to C14, C17 to C15, C14 to C16, C15 to C17, C3 to C2, C5 to C3, C7 to C4, D4 to D10, D6 to D11, D8 to D12, D10 to D13, D12 to D14, D17 to D16, D19 to D17, D21 to D18, D23 to D19, D3 to D2, D25 to D20, D27 to D21, D29 to D22, D16 to D23, D18 to D24, D20 to D25, D22 to D26, D24 to D27, D26 to D28, D28 to D29, D5 to D3, D7 to D4, D41 to D40, D43 to D41, D45 to D42, D47 to D43, D49 to D44, D51 to D45, D52 to D46, D40 to D47, D42 to D48, D44 to D49, D9 to D5, D46 to D50, D48 to D51, D50 to D52, D55 to D54, D57 to D55, D59 to D56, D61 to D57, D63 to D58, D65 to D59, D11 to D6, D66 to D60, D54 to D61, D56 to D62, D58 to D63, D60 to D64, D62 to D65, D64 to D66, D69 to D68, D71 to D69, D13 to D7, D73 to D70, D75 to D71, D77 to D72, D79 to D73, D81 to D74, D68 to D75, D70 to D76, D72 to D77, D74 to D78, D76 to D79, D14 to D8, D78 to D80, D80 to D81, D2 to D9, J2 to J1, J1 to J2, R4 to R1, R12 to R10, R14 to R11, R10 to R12, R8 to R13, R9 to R14, R6 to R2, R1 to R3, R2 to R4, R3 to R5, R5 to R6, R11 to R8, R13 to R9, SW3 to SW10, SW5 to SW11, SW7 to SW12, SW9 to SW13, SW11 to SW14, SW13 to SW15, SW18 to SW17, SW20 to SW18, SW22 to SW19, SW24 to SW20, SW26 to SW21, SW28 to SW22, SW30 to SW23, SW17 to SW24, SW19 to SW25, SW21 to SW26, SW23 to SW27, SW25 to SW28, SW27 to SW29, SW4 to SW3, SW29 to SW30, SW6 to SW4, SW42 to SW41, SW44 to SW42, SW46 to SW43, SW48 to SW44, SW50 to SW45, SW52 to SW46, SW53 to SW47, SW41 to SW48, SW43 to SW49, SW8 to SW5, SW45 to SW50, SW47 to SW51, SW49 to SW52, SW51 to SW53, SW56 to SW55, SW58 to SW56, SW60 to SW57, SW62 to SW58, SW64 to SW59, SW10 to SW6, SW66 to SW60, SW67 to SW61, SW55 to SW62, SW57 to SW63, SW59 to SW64, SW61 to SW65, SW63 to SW66, SW65 to SW67, SW70 to SW69, SW12 to SW7, SW72 to SW70, SW74 to SW71, SW76 to SW72, SW78 to SW73, SW80 to SW74, SW82 to SW75, SW69 to SW76, SW71 to SW77, SW73 to SW78, SW75 to SW79, SW14 to SW8, SW77 to SW80, SW79 to SW81, SW81 to SW82, SW15 to SW9, U3 to U2, U2 to U3, U7 to U5, U8 to U6, U5 to U7, U6 to U8
Connections:
- C10 pad 2: +3V3 -> /VCAP1
- C6 pad 1: /OSC_OUT -> GND
- C6 pad 2: GND -> +3V3
- C8 pad 1: GND -> /OSC_OUT
- C8 pad 2: +3V3 -> GND
- D14 pad 1: /C13 -> /C14
- D33 pad 1: /C3 -> /C5
- D34 pad 1: /C4 -> /C9
- D35 pad 1: /C5 -> /C10
- D36 pad 1: /C6 -> /C12
- D37 pad 1: /C7 -> /C13
- D38 pad 1: /C8 -> /C14
- D50 pad 1: /C11 -> /C12
- D51 pad 1: /C12 -> /C13
- D52 pad 1: /C13 -> /C14
- D65 pad 1: /C12 -> /C13
- D66 pad 1: /C13 -> /C14
Other:
- board size 304.8 x 123.8 mm -> 304.8 x 125.7 mm

Commit message: Places gesture sensors onto board layout for cherry mx pcb mounted keyboard.
Parts:
- moved U6 426.0 mm to (294.3, 66.7)
- moved C15 421.3 mm to (298.4, 66.0), turned to 90 degrees
- moved R11 411.9 mm to (288.9, 64.8)
- moved R10 411.8 mm to (288.9, 68.6)
- moved C13 341.9 mm to (127.0, 66.0), turned to 90 degrees
- moved U5 340.2 mm to (208.6, 66.7)
- moved C14 340.0 mm to (212.7, 66.0), turned to 90 degrees
- moved U4 336.9 mm to (122.9, 66.7)
- moved R9 330.6 mm to (203.2, 64.8)
- moved R8 330.4 mm to (203.2, 68.6)
- moved J2 288.3 mm to (37.1, 47.0), turned to 180 degrees
- moved R7 275.9 mm to (117.5, 64.8)
- moved R6 273.2 mm to (117.5, 68.6)
- moved U2 258.4 mm to (37.1, 66.7)
- moved C12 254.0 mm to (41.3, 66.0), turned to 90 degrees
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
Commit message: Changes bypass capacitors for the stm32f413 to 0603 on the cherry mx pcb mounted keyboard. Also the sensors were not centered in between row 0 and 1 so that was fixed. Y position not 2.6375in
Parts:
- C1, C10, C4: footprint Capacitor_SMD:C_0805_2012Metric -> Capacitor_SMD:C_0603_1608Metric
- C2, C3, C5, C6, C7, C8: footprint Capacitor_SMD:C_0805_2012Metric -> Capacitor_SMD:C_0603_1608Metric; moved to B.Cu
- C9, D82, J1, JP1, R12, R13, R14, SW1, U1, Y1: moved to B.Cu
- moved R12 324.9 mm to (165.7, 50.2), turned to 270 degrees
- moved D82 301.2 mm to (165.7, 45.7), turned to 270 degrees
- moved J1 263.4 mm to (61.0, 52.7), turned to 270 degrees
- moved C1 249.7 mm to (96.5, -10.8)
- moved C4 249.7 mm to (109.9, -4.45)
- moved C11 243.4 mm to (77.5, 61.6)
- moved SW1 226.0 mm to (122.9, 47.6)
- moved U8 222.7 mm to (37.1, 54.6), turned to 180 degrees
- moved C9 222.0 mm to (122.9, 50.8)
- moved C16 219.6 mm to (21.0, 61.6)
- moved U7 209.1 mm to (21.0, 67.0), turned to 180 degrees
- moved C17 208.3 mm to (21.0, 72.4)
- moved R14 194.9 mm to (38.7, 47.0), turned to 90 degrees
- moved R13 190.9 mm to (35.6, 47.0), turned to 90 degrees
- moved JP1 183.3 mm to (80.0, 52.7), turned to 90 degrees
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
Commit message: Places all components onto the board for the cherry mx pcb mounted keyboard.
Parts:
- C1, C4: moved to B.Cu
- moved C1 105.7 mm to (32.5, 73.3), turned to 45 degrees
- moved C4 91.7 mm to (45.7, 61.2), turned to 315 degrees
- moved C5 44.8 mm to (36.2, 74.9)
- moved C6 43.6 mm to (38.1, 74.9)
Other:
- net class Default: trace_width 0.25 -> 0.4; via_dia 0.8 -> 0.6; via_drill 0.4 -> 0.3
Changed lines of the file:
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@@
   )
   (setup
-    (last_trace_width 0.25)
+    (last_trace_width 0.4)
     (trace_clearance 0.2)
     (zone_clearance 0.508)
     (zone_45_only no)
     (trace_min 0.2)
-    (via_size 0.8)
-    (via_drill 0.4)
+    (via_size 0.6)
+    (via_drill 0.3)
     (via_min_size 0.4)
     (via_min_drill 0.3)
@@
   (net_class Default "This is the default net class."
     (clearance 0.2)
-    (trace_width 0.25)
-    (via_dia 0.8)
-    (via_drill 0.4)
+    (trace_width 0.4)
+    (via_dia 0.6)
+    (via_drill 0.3)
     (uvia_dia 0.3)
     (uvia_drill 0.1)
@@
     (tags capacitor)
     (attr smd)
-    (fp_text reference C8 (at 0 1.43 45) (layer B.SilkS)
+    (fp_text reference C8 (at 0 1.43 45) (layer B.SilkS) hide
       (effects (font (size 1 1) (thickness 0.15)) (justify mirror))
     )
@@
     (tags capacitor)
     (attr smd)
-    (fp_text reference C7 (at 0 1.43 45) (layer B.SilkS)
+    (fp_text reference C7 (at 0 1.43 45) (layer B.SilkS) hide
       (effects (font (size 1 1) (thickness 0.15)) (justify mirror))
     )
@@
     )
   )
-  (module Capacitor_SMD:C_0603_1608Metric (layer F.Cu)
-    (at 109.855 -4.445 90)
+  (module Capacitor_SMD:C_0603_1608Metric (layer B.Cu)
+    (at 45.72 61.1505 315)
     (descr "Capacitor SMD 0603 (1608 Metric), square (rectangular) end terminal, IPC_7351 nominal, (Body size source: http://www.tortai-tech.com/upload/download/2011102023233369053.pdf), generated with kicad-footprint-generator")
     (tags capacitor)
     (attr smd)
-    (fp_text reference C4 (at 0 -1.43 90) (layer F.SilkS)
-      (effects (font (size 1 1) (thickness 0.15)))
+    (fp_text reference C4 (at 0 1.43 315) (layer B.SilkS) hide
+      (effects (font (size 1 1) (thickness 0.15)) (justify mirror))
     )
-    (fp_text value 4.7u (at 0 1.43 90) (layer F.Fab)
-      (effects (font (size 1 1) (thickness 0.15)))
+    (fp_text value 4.7u (at 0 -1.43 315) (layer B.Fab)
+      (effects (font (size 1 1) (thickness 0.15)) (justify mirror))
     )
-    (fp_text user %R (at 0 0 90) (layer F.Fab)
-      (effects (font (size 0.4 0.4) (thickness 0.06)))
+    (fp_text user %R (at 0 0 315) (layer B.Fab)
+      (effects (font (size 0.4 0.4) (thickness 0.06)) (justify mirror))
     )
-    (fp_line (start 1.48 0.73) (end -1.48 0.73) (layer F.CrtYd) (width 0.05))
-    (fp_line (start 1.48 -0.73) (end 1.48 0.73) (layer F.CrtYd) (width 0.05))
-    (fp_line (start -1.48 -0.73) (end 1.48 -0.73) (layer F.CrtYd) (width 0.05))
-    (fp_line (start -1.48 0.73) (end -1.48 -0.73) (layer F.CrtYd) (width 0.05))
-    (fp_line (start -0.162779 0.51) (end 0.162779 0.51) (layer F.SilkS) (width 0.12))
-    (fp_line (start -0.162779 -0.51) (end 0.162779 -0.51) (layer F.SilkS) (width 0.12))
-    (fp_line (start 0.8 0.4) (end -0.8 0.4) (layer F.Fab) (width 0.1))
-    (fp_line (start 0.8 -0.4) (end 0.8 0.4) (layer F.Fab) (width 0.1))
-    (fp_line (start -0.8 -0.4) (end 0.8 -0.4) (layer F.Fab) (width 0.1))
-    (fp_line (start -0.8 0.4) (end -0.8 -0.4) (layer F.Fab) (width 0.1))
-    (pad 2 smd roundrect (at 0.7875 0 90) (size 0.875 0.95) (layers F.Cu F.Paste F.Mask) (roundrect_rratio 0.25)
+    (fp_line (start 1.48 -0.73) (end -1.48 -0.73) (layer B.CrtYd) (width 0.05))
+    (fp_line (start 1.48 0.73) (end 1.48 -0.73) (layer B.CrtYd) (width 0.05))
+    (fp_line (start -1.48 0.73) (end 1.48 0.73) (layer B.CrtYd) (width 0.05))
+    (fp_line (start -1.48 -0.73) (end -1.48 0.73) (layer B.CrtYd) (width 0.05))
+    (fp_line (start -0.162779 -0.51) (end 0.162779 -0.51) (layer B.SilkS) (width 0.12))
+    (fp_line (start -0.162779 0.51) (end 0.162779 0.51) (layer B.SilkS) (width 0.12))
+    (fp_line (start 0.8 -0.4) (end -0.8 -0.4) (layer B.Fab) (width 0.1))
+    (fp_line (start 0.8 0.4) (end 0.8 -0.4) (layer B.Fab) (width 0.1))
+    (fp_line (start -0.8 0.4) (end 0.8 0.4) (layer B.Fab) (width 0.1))
+    (fp_line (start -0.8 -0.4) (end -0.8 0.4) (layer B.Fab) (width 0.1))
+    (pad 2 smd roundrect (at 0.7875 0 315) (size 0.875 0.95) (layers B.Cu B.Paste B.Mask) (roundrect_rratio 0.25)
       (net 82 +3V3))
-    (pad 1 smd roundrect (at -0.7875 0 90) (size 0.875 0.95) (layers F.Cu F.Paste F.Mask) (roundrect_rratio 0.25)
+    (pad 1 smd roundrect (at -0.7875 0 315) (size 0.875 0.95) (layers B.Cu B.Paste B.Mask) (roundrect_rratio 0.25)
       (net 73 GND))
     (model ${KISYS3DMOD}/Capacitor_SMD.3dshapes/C_0603_1608Metric.wrl
@@
     )
   )
-  (module Capacitor_SMD:C_0603_1608Metric (layer F.Cu)
-    (at 96.52 -10.795 180)
+  (module Capacitor_SMD:C_0603_1608Metric (layer B.Cu)
+    (at 32.512 73.279 45)
     (descr "Capacitor SMD 0603 (1608 Metric), square (rectangular) end terminal, IPC_7351 nominal, (Body size source: http://www.tortai-tech.com/upload/download/2011102023233369053.pdf), generated with kicad-footprint-generator")
     (tags capacitor)
     (attr smd)
-    (fp_text reference C1 (at 0 -1.43) (layer F.SilkS)
-      (effects (font (size 1 1) (thickness 0.15)))
+    (fp_text reference C1 (at 0 1.43 45) (layer B.SilkS) hide
+      (effects (font (size 1 1) (thickness 0.15)) (justify mirror))
     )
-    (fp_text value 0.1u (at 0 1.43) (layer F.Fab)
-      (effects (font (size 1 1) (thickness 0.15)))
+    (fp_text value 0.1u (at 0 -1.43 45) (layer B.Fab)
+      (effects (font (size 1 1) (thickness 0.15)) (justify mirror))
     )
-    (fp_text user %R (at 0 0) (layer F.Fab)
-      (effects (font (size 0.4 0.4) (thickness 0.06)))
+    (fp_text user %R (at 0 0 45) (layer B.Fab)
+      (effects (font (size 0.4 0.4) (thickness 0.06)) (justify mirror))
     )
-    (fp_line (start 1.48 0.73) (end -1.48 0.73) (layer F.CrtYd) (width 0.05))
-    (fp_line (start 1.48 -0.73) (end 1.48 0.73) (layer F.CrtYd) (width 0.05))
-    (fp_line (start -1.48 -0.73) (end 1.48 -0.73) (layer F.CrtYd) (width 0.05))
-    (fp_line (start -1.48 0.73) (end -1.48 -0.73) (layer F.CrtYd) (width 0.05))
-    (fp_line (start -0.162779 0.51) (end 0.162779 0.51) (layer F.SilkS) (width 0.12))
-    (fp_line (start -0.162779 -0.51) (end 0.162779 -0.51) (layer F.SilkS) (width 0.12))
-    (fp_line (start 0.8 0.4) (end -0.8 0.4) (layer F.Fab) (width 0.1))
-    (fp_line (start 0.8 -0.4) (end 0.8 0.4) (layer F.Fab) (width 0.1))
-    (fp_line (start -0.8 -0.4) (end 0.8 -0.4) (layer F.Fab) (width 0.1))
-    (fp_line (start -0.8 0.4) (end -0.8 -0.4) (layer F.Fab) (width 0.1))
-    (pad 2 smd roundrect (at 0.7875 0 180) (size 0.875 0.95) (layers F.Cu F.Paste F.Mask) (roundrect_rratio 0.25)
+    (fp_line (start 1.48 -0.73) (end -1.48 -0.73) (layer B.CrtYd) (width 0.05))
+    (fp_line (start 1.48 0.73) (end 1.48 -0.73) (layer B.CrtYd) (width 0.05))
+    (fp_line (start -1.48 0.73) (end 1.48 0.73) (layer B.CrtYd) (width 0.05))
+    (fp_line (start -1.48 -0.73) (end -1.48 0.73) (layer B.CrtYd) (width 0.05))
+    (fp_line (start -0.162779 -0.51) (end 0.162779 -0.51) (layer B.SilkS) (width 0.12))
+    (fp_line (start -0.162779 0.51) (end 0.162779 0.51) (layer B.SilkS) (width 0.12))
+    (fp_line (start 0.8 -0.4) (end -0.8 -0.4) (layer B.Fab) (width 0.1))
+    (fp_line (start 0.8 0.4) (end 0.8 -0.4) (layer B.Fab) (width 0.1))
+    (fp_line (start -0.8 0.4) (end 0.8 0.4) (layer B.Fab) (width 0.1))
+    (fp_line (start -0.8 -0.4) (end -0.8 0.4) (layer B.Fab) (width 0.1))
+    (pad 2 smd roundrect (at 0.7875 0 45) (size 0.875 0.95) (layers B.Cu B.Paste B.Mask) (roundrect_rratio 0.25)
       (net 82 +3V3))
-    (pad 1 smd roundrect (at -0.7875 0 180) (size 0.875 0.95) (layers F.Cu F.Paste F.Mask) (roundrect_rratio 0.25)
+    (pad 1 smd roundrect (at -0.7875 0 45) (size 0.875 0.95) (layers B.Cu B.Paste B.Mask) (roundrect_rratio 0.25)
       (net 73 GND))
     (model ${KISYS3DMOD}/Capacitor_SMD.3dshapes/C_0603_1608Metric.wrl
@@
       (effects (font (size 1 1) (thickness 0.15)))
     )
-    (fp_text value APDS-9960 (at 0 0) (layer F.SilkS)
+    (fp_text value APDS-9960 (at 0 0) (layer F.SilkS) hide
       (effects (font (size 1 1) (thickness 0.15)))
     )
@@
       (effects (font (size 1 1) (thickness 0.15)))
     )
-    (fp_text value APDS-9960 (at 0 0) (layer F.SilkS)
+    (fp_text value APDS-9960 (at 0 0) (layer F.SilkS) hide
       (effects (font (size 1 1) (thickness 0.15)))
     )
@@
   )
   (module Capacitor_SMD:C_0603_1608Metric (layer B.Cu)
-    (at -6.985 62.865 90)
+    (at 36.195 74.93 90)
     (descr "Capacitor SMD 0603 (1608 Metric), square (rectangular) end terminal, IPC_7351 nominal, (Body size source: http://www.tortai-tech.com/upload/download/2011102023233369053.pdf), generated with kicad-footprint-generator")
     (tags capacitor)
     (attr smd)
-    (fp_text reference C5 (at 0 1.43 90) (layer B.SilkS)
+    (fp_text reference C5 (at 0 1.43 90) (layer B.SilkS) hide
       (effects (font (size 1 1) (thickness 0.15)) (justify mirror))
     )
@@
   )
   (module Capacitor_SMD:C_0603_1608Metric (layer B.Cu)
-    (at -3.81 62.865 90)
+    (at 38.1 74.93 90)
     (descr "Capacitor SMD 0603 (1608 Metric), square (rectangular) end terminal, IPC_7351 nominal, (Body size source: http://www.tortai-tech.com/upload/download/2011102023233369053.pdf), generated with kicad-footprint-generator")
     (tags capacitor)
     (attr smd)
-    (fp_text reference C6 (at 0 1.43 90) (layer B.SilkS)
+    (fp_text reference C6 (at 0 1.43 90) (layer B.SilkS) hide
       (effects (font (size 1 1) (thickness 0.15)) (justify mirror))
     )
