File: hardware/keyboard-cherry-mx-pcb-mounted/keyboard-cherry-mx-pcb-mounted.kicad_pcb (KiCad board)
At the start: 2 copper layers, 304.8 x 125.7 mm, 207 parts, among them J1 SWDConn, J2 USB_C_Receptacle_USB2.0, SW1 RST, SW10 F8, SW11 F9, SW12 F10, SW13 F11, SW14 F12, SW15 Delete, SW16 `, SW17 1, SW18 2, SW19 3, SW2 ESC, SW20 4, SW21 5, SW22 6, SW23 7, SW24 8, SW25 9, SW26 0, SW27 -, SW28 =, SW29 Backspace, SW3 F1, SW30 Home, SW31 Ctrl, SW32 Workspace, SW33 Alt, SW34 Space, SW35 Alt, SW36 Ctrl, SW37 Left Arrow, SW38 Down Arrow, SW39 Right Arrow, SW4 F2, SW40 LShift, SW41 z, SW42 x, SW43 c, SW44 v, SW45 b, SW46 n, SW47 m, SW48 ,, SW49 ., SW5 F3, SW50 /, SW51 RShift, SW52 Up Arrow, SW53 End, SW54 Caps lock, SW55 a, SW56 s, SW57 d, SW58 f, SW59 g, SW6 F4, SW60 h, SW61 j, SW62 k, SW63 l, SW64 ;, SW65 ', SW66 Enter, SW67 PgDn, SW68 Tab, SW69 q, SW7 F5, SW70 w, SW71 e, SW72 r, SW73 t, SW74 y, SW75 u, SW76 i, SW77 o, SW78 p, SW79 [, SW8 F6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

Commit message: Starts routing all traces for the cherry mx pcb mounted keyboard.
Routing:
- net /R1: track 0.00 -> 287.9 mm
- net /R0: track 0.00 -> 285.8 mm
- net /R5: track 0.00 -> 285.5 mm
- net /R2: track 0.00 -> 281.0 mm
- net /R3: track 0.00 -> 280.7 mm
- net /R4: track 0.00 -> 274.9 mm
- net /C12: track 0.00 -> 82.4 mm
- net Net-(D50-Pad2): track 0.00 -> 8.38 mm
- net Net-(D37-Pad2): track 0.00 -> 8.38 mm
- net Net-(D36-Pad2): track 0.00 -> 8.38 mm
- net Net-(D35-Pad2): track 0.00 -> 8.38 mm
- net Net-(D47-Pad2): track 0.00 -> 8.38 mm
- net Net-(D51-Pad2): track 0.00 -> 8.38 mm
- net Net-(D65-Pad2): track 0.00 -> 8.38 mm
- net Net-(D64-Pad2): track 0.00 -> 8.38 mm
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
Commit message: Places traces at optimal location. Need to wire up the rest of the columns.
Parts:
- moved C2 4.94 mm to (38.4, 55.4), turned to 225 degrees
- moved U8 0.48 mm to (37.1, 54.1)
- moved C15 0.43 mm to (298.4, 66.5)
- moved C12 0.43 mm to (41.3, 66.5)
- moved C13 0.43 mm to (127.0, 66.5)
- moved C14 0.43 mm to (212.7, 66.5)
- moved C7 0.31 mm to (48.9, 67.9)
- moved C8 0.21 mm to (42.4, 74.4)
- moved Y1 0.07 mm to (45.6, 71.1)
Routing:
- net GND: track 0.00 -> 519.4 mm, vias 0 -> 20
- net +3V3: track 0.00 -> 493.8 mm, vias 0 -> 22
- net /C10: track 0.00 -> 353.5 mm, vias 0 -> 2
- net /C11: track 0.00 -> 317.7 mm, vias 0 -> 2
- net /C12: track 82.4 -> 378.2 mm, vias 0 -> 2
- net /C5: track 0.00 -> 251.1 mm, vias 0 -> 4
- net Net-(R10-Pad2): track 0.00 -> 223.8 mm, vias 0 -> 3
- net Net-(R11-Pad2): track 0.00 -> 216.5 mm
- net /C4: track 0.00 -> 203.6 mm, vias 0 -> 4
- net /C2: track 0.00 -> 193.4 mm, vias 0 -> 4
- net /C9: track 0.00 -> 184.1 mm, vias 0 -> 2
- net /C3: track 0.00 -> 182.1 mm, vias 0 -> 4
- net /C1: track 0.00 -> 177.4 mm, vias 0 -> 2
- net /C0: track 0.00 -> 164.3 mm, vias 0 -> 2
- net /C8: track 0.00 -> 144.5 mm, vias 0 -> 2
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Other:
- net class Default: clearance 0.2 -> 0.127; trace_width 0.4 -> 0.15
- rule trace_clearance: 0.2 -> 0.127
- rule trace_min: 0.2 -> 0.127
- rule via_min_size: 0.4 -> 0.6

Commit message: Finishes tracing for cherry mx pcb mounted keyboard.
Routing:
- net /C14: track 137.8 -> 434.6 mm, vias 1 -> 4
- net /C13: track 108.0 -> 379.8 mm, vias 1 -> 4
- net /PB15: track 33.5 -> 283.4 mm, vias 2 -> 7
- net /C9: track 184.1 -> 364.7 mm, vias 2 -> 6
- net /C8: track 144.5 -> 303.8 mm, vias 2 -> 6
- net /PB14: track 33.0 -> 190.4 mm, vias 2 -> 3
- net /C7: track 143.8 -> 296.1 mm, vias 2 -> 4
- net /C6: track 143.2 -> 274.6 mm, vias 2 -> 4
- net /PB13: track 32.3 -> 103.8 mm, vias 2 -> 3
- net Net-(D82-Pad2): track 0.00 -> 2.57 mm
- net /C2: track 193.4 -> 195.7 mm
- net Net-(R6-Pad2): vias 3 -> 4

Commit message: Adds mounting holes to the cherry mx pcb mounted keyboard.
Parts:
- added H1: M2, MountingHole:MountingHole_2.2mm_M2, F.Cu at (156.2, 91.0)
- added H10: M2, MountingHole:MountingHole_2.2mm_M2, F.Cu at (112.7, 159.0)
- added H2: M2, MountingHole:MountingHole_2.2mm_M2, F.Cu at (274.7, 139.0)
- added H3: M2, MountingHole:MountingHole_2.2mm_M2, F.Cu at (198.9, 119.8)
- added H4: M2, MountingHole:MountingHole_2.2mm_M2, F.Cu at (292.7, 120.0)
- added H5: M2, MountingHole:MountingHole_2.2mm_M2, F.Cu at (274.7, 67.1)
- added H6: M2, MountingHole:MountingHole_2.2mm_M2, F.Cu at (65.7, 120.0)
- added H7: M2, MountingHole:MountingHole_2.2mm_M2, F.Cu at (17.7, 138.0)
- added H8: M2, MountingHole:MountingHole_2.2mm_M2, F.Cu at (39.7, 101.0)
- added H9: M2, MountingHole:MountingHole_2.2mm_M2, F.Cu at (102.7, 67.1)

Commit message: Adds labels for each key and creates gerber files.
Parts:
- added G***: LOGO, Sij_Special:SJW_Logo_25x25mm, F.Cu at (165.4, 67.0)
- SW10: value F8 -> f8
- SW11: value F9 -> f9
- SW12: value F10 -> f10
- SW13: value F11 -> f11
- SW14: value F12 -> f12
- SW15: value Delete -> delete
- SW2: value ESC -> esc
- SW29: value Backspace -> backspace
- SW3: value F1 -> f1
- SW30: value Home -> home
- SW31, SW36: value Ctrl -> ctrl
- SW32: value Workspace -> workspace
- SW33, SW35: value Alt -> alt
- SW34: value Space -> space
- SW37: value Left Arrow -> left
- SW38: value Down Arrow -> down
- SW39: value Right Arrow -> right
- SW4: value F2 -> f2
- SW40: value LShift -> lshift
- SW5: value F3 -> f3
- SW51: value RShift -> rshift
- SW52: value Up Arrow -> up
- SW53: value End -> end
- SW54: value Caps lock -> caps lock
- SW6: value F4 -> f4
- SW66: value Enter -> enter
- SW67: value PgDn -> pgdn
- SW68: value Tab -> tab
- SW7: value F5 -> f5
- SW8: value F6 -> f6
- SW82: value PgUp -> pgup
- SW9: value F7 -> f7
Other:
- board text added: "Blossum v1.0 Spring 2020 Sijin Woo"
